File: Hardware/PCB/PCB.kicad_pcb (KiCad board)
At the start: 2 copper layers, 324.1 x 114.5 mm, 163 parts, among them U1 ESP32-S3-DevKitC

Commit message: finished tracing
Routing:
- net /row4: track 0.00 -> 290.3 mm
- net /row3: track 0.00 -> 262.7 mm
- net /row5: track 283.4 -> 323.1 mm
- net /col8: track 167.8 -> 188.8 mm
- net Net-(D65-A): track 0.00 -> 6.32 mm
- net Net-(D35-A): track 0.00 -> 6.32 mm
- net Net-(D17-A): track 0.00 -> 6.32 mm
- net Net-(D59-A): track 0.00 -> 6.32 mm
- net Net-(D53-A): track 0.00 -> 6.32 mm
- net Net-(D41-A): track 0.00 -> 6.32 mm
- net Net-(D29-A): track 0.00 -> 6.32 mm
- net Net-(D23-A): track 0.00 -> 6.32 mm
- net Net-(D74-A): track 0.00 -> 6.32 mm
- net Net-(D70-A): track 0.00 -> 6.32 mm
- net Net-(D47-A): track 0.00 -> 6.32 mm
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
Commit message: sch changes
Parts:
- added H1: Stabilizer 6.5u, PCM_Mounting_Keyboard_Stabilizer:Stabilizer_Cherry_MX_6.25u, F.Cu at (172.2, 146.5)
- added H2: Stabilizer 2u, PCM_Mounting_Keyboard_Stabilizer:Stabilizer_Cherry_MX_2.00u, F.Cu at (291.3, 127.4)
- added H3: Stabilizer 2u, PCM_Mounting_Keyboard_Stabilizer:Stabilizer_Cherry_MX_2.00u, F.Cu at (115.2, 232.8)
- added H4: Stabilizer 2u, PCM_Mounting_Keyboard_Stabilizer:Stabilizer_Cherry_MX_2.00u, F.Cu at (115.2, 252.6)
Connections:
- net /col0 renamed /a
- net /col1 renamed /b
- net /col10 renamed /k
- net /col11 renamed /l
- net /col12 renamed /m
- net /col13 renamed /n
- net /col14 renamed /o
- net /col2 renamed /c
- net /col3 renamed /d
- net /col4 renamed /e
- net /col5 renamed /f
- net /col6 renamed /g
- net /col7 renamed /h
- net /col8 renamed /i
- net /col9 renamed /j
- net /row0 renamed /1
- net /row1 renamed /2
- net /row2 renamed /3
- net /row3 renamed /4
- net /row4 renamed /5
- net /row5 renamed /6
Other:
- board text added: "Keyboard V1.0"
- board text added: "github.com/FelTell"

Commit message: added tracks
Parts:
- S3: footprint PCM_Switch_Keyboard_Cherry_MX:SW_Cherry_MX_PCB_1.50u -> PCM_Switch_Keyboard_Cherry_MX:SW_Cherry_MX_PCB_1.25u
- S30: footprint PCM_Switch_Keyboard_Cherry_MX:SW_Cherry_MX_PCB_6.25u -> PCM_Switch_Keyboard_Cherry_MX:SW_Cherry_MX_PCB_1.00u
- S4: footprint PCM_Switch_Keyboard_Cherry_MX:SW_Cherry_MX_PCB_1.75u -> PCM_Switch_Keyboard_Cherry_MX:SW_Cherry_MX_PCB_1.25u
- S42: footprint PCM_Switch_Keyboard_Cherry_MX:SW_Cherry_MX_PCB_1.00u -> PCM_Switch_Keyboard_Cherry_MX:SW_Cherry_MX_PCB_6.25u
- S5: footprint PCM_Switch_Keyboard_Cherry_MX:SW_Cherry_MX_PCB_1.25u -> PCM_Switch_Keyboard_Cherry_MX:SW_Cherry_MX_PCB_1.50u
- S6: footprint PCM_Switch_Keyboard_Cherry_MX:SW_Cherry_MX_PCB_1.25u -> PCM_Switch_Keyboard_Cherry_MX:SW_Cherry_MX_PCB_1.75u
- S60, S71: footprint PCM_Switch_Keyboard_Cherry_MX:SW_Cherry_MX_PCB_1.00u -> PCM_Switch_Keyboard_Cherry_MX:SW_Cherry_MX_PCB_1.25u
- S73: footprint PCM_Switch_Keyboard_Cherry_MX:SW_Cherry_MX_PCB_1.00u -> PCM_Switch_Keyboard_Cherry_MX:SW_Cherry_MX_PCB_2.75u
- S74: footprint PCM_Switch_Keyboard_Cherry_MX:SW_Cherry_MX_PCB_2.75u -> PCM_Switch_Keyboard_Cherry_MX:SW_Cherry_MX_PCB_2.25u
- S75: footprint PCM_Switch_Keyboard_Cherry_MX:SW_Cherry_MX_PCB_1.00u -> PCM_Switch_Keyboard_Cherry_MX:SW_Cherry_MX_PCB_2.00u
- S76: footprint PCM_Switch_Keyboard_Cherry_MX:SW_Cherry_MX_PCB_1.00u -> PCM_Switch_Keyboard_Cherry_MX:SW_Cherry_MX_PCB_1.50u
- S77: footprint PCM_Switch_Keyboard_Cherry_MX:SW_Cherry_MX_PCB_2.00u -> PCM_Switch_Keyboard_Cherry_MX:SW_Cherry_MX_PCB_1.00u
- S78: footprint PCM_Switch_Keyboard_Cherry_MX:SW_Cherry_MX_PCB_1.50u -> PCM_Switch_Keyboard_Cherry_MX:SW_Cherry_MX_PCB_1.00u
- S79: footprint PCM_Switch_Keyboard_Cherry_MX:SW_Cherry_MX_PCB_2.25u -> PCM_Switch_Keyboard_Cherry_MX:SW_Cherry_MX_PCB_1.00u
- moved H3 224.7 mm to (292.9, 95.2)
- moved H4 221.4 mm to (288.1, 114.3)
- moved S36 126.1 mm to (152.4, 57.1)
- moved D36 125.6 mm to (161.1, 57.1)
- moved S30 115.3 mm to (133.3, 38.1)
- moved D30 115.0 mm to (142.1, 38.1)
- moved S54 113.4 mm to (219.1, 76.2)
- moved D54 112.8 mm to (227.8, 76.2)
- moved S42 92.2 mm to (169.1, 133.3)
- moved D35 90.2 mm to (161.1, 38.1)
- moved S35 90.2 mm to (152.4, 38.1)
- moved S48 90.1 mm to (195.3, 114.3)
- moved D48 89.4 mm to (204.0, 114.3)
- moved S60 87.5 mm to (240.5, 133.3)
- moved D60 84.5 mm to (251.6, 133.3)
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Connections:
- net GND renamed Net-(U1-GND-Pad22)
- D10 pad 1: /4 -> /5
- D11 pad 1: /5 -> /3
- D12 pad 1: /6 -> /4
- D15 pad 1: /3 -> /6
- D16 pad 1: /4 -> /5
- D17 pad 1: /5 -> /3
- D18 pad 1: /6 -> /4
- D21 pad 1: /3 -> /6
- D22 pad 1: /4 -> /5
- D23 pad 1: /5 -> /3
- D24 pad 1: /6 -> /4
- D27 pad 1: /3 -> /5
- D28 pad 1: /4 -> /3
- D29 pad 1: /5 -> /4
- D3 pad 1: /3 -> /6
- D30 pad 1: /6 -> /1
- D31 pad 1: /1 -> /2
- D32 pad 1: /2 -> /5
- D35 pad 1: /5 -> /1
- D36 pad 1: /6 -> /2
- D37 pad 1: /1 -> /5
- D38 pad 1: /2 -> /3
- D39 pad 1: /3 -> /4
- D4 pad 1: /4 -> /5
- D40 pad 1: /4 -> /1
- D41 pad 1: /5 -> /2
- D43 pad 1: /1 -> /5
- D44 pad 1: /2 -> /3
- D45 pad 1: /3 -> /4
- D46 pad 1: /4 -> /1
- D47 pad 1: /5 -> /2
- D48 pad 1: /6 -> /5
- D49 pad 1: /1 -> /3
- D5 pad 1: /5 -> /3
- D50 pad 1: /2 -> /4
- D51 pad 1: /3 -> /1
- D52 pad 1: /4 -> /2
- D54 pad 1: /6 -> /3
- D55 pad 1: /1 -> /4
- D56 pad 1: /2 -> /1
- D57 pad 1: /3 -> /2
- D58 pad 1: /4 -> /5
- D59 pad 1: /5 -> /3
- D6 pad 1: /6 -> /4
- D61 pad 1: /1 -> /4
- D62 pad 1: /2 -> /1
- D63 pad 1: /3 -> /2
- D64 pad 1: /4 -> /5
- D65 pad 1: /5 -> /3
- D66 pad 1: /1 -> /6
- D67 pad 1: /2 -> /4
- D68 pad 1: /3 -> /1
- D69 pad 1: /4 -> /2
- D70 pad 1: /5 -> /3
- D71 pad 1: /1 -> /6
- D72 pad 1: /2 -> /1
- D73 pad 1: /3 -> /5
- D74 pad 1: /5 -> /4
- D75 pad 1: /1 -> /2
- D76 pad 1: /1 -> /3
- D77 pad 1: /2 -> /1
- D78 pad 1: /3 -> /6
- D79 pad 1: /4 -> /6
- D9 pad 1: /3 -> /6
- S30 pad 1: /e -> /f
- S35 pad 1: /f -> /g
- S36 pad 1: /f -> /g
- S40 pad 1: /g -> /h
- S41 pad 1: /g -> /h
- S46 pad 1: /h -> /i
- S47 pad 1: /h -> /i
- S48 pad 1: /h -> /i
- S51 pad 1: /i -> /j
- S52 pad 1: /i -> /j
- S53 pad 1: /i -> /j
- S54 pad 1: /i -> /j
- S56 pad 1: /j -> /k
- S57 pad 1: /j -> /k
- S58 pad 1: /j -> /k
- S59 pad 1: /j -> /k
- S60 pad 1: /j -> /i
- S62 pad 1: /k -> /l
- S63 pad 1: /k -> /l
- S64 pad 1: /k -> /l
- S65 pad 1: /k -> /l
- S66 pad 1: /l -> /j
- S68 pad 1: /l -> /m
- S69 pad 1: /l -> /m
- S70 pad 1: /l -> /m
- S71 pad 1: /m -> /k
- S72 pad 1: /m -> /n
- S74 pad 1: /m -> /o
- S75 pad 1: /n -> /o
- S78 pad 1: /o -> /l
- S79 pad 2: Net-(D79-A) -> Net-(D80-A)
- S80 pad 1: /o -> /m
- S80 pad 2: Net-(D80-A) -> Net-(D79-A)
- U1 pad 10: unconnected-(U1-GPIO17/ADC2_CH6-Pad10) -> /m
- U1 pad 11: unconnected-(U1-GPIO18/ADC2_CH7-Pad11) -> /n
- U1 pad 12: unconnected-(U1-GPIO8/ADC1_CH7-Pad12) -> /d
- U1 pad 15: unconnected-(U1-GPIO9/ADC1_CH8-Pad15) -> /e
- U1 pad 16: unconnected-(U1-GPIO10/ADC1_CH9-Pad16) -> /f
- U1 pad 17: unconnected-(U1-GPIO11/ADC2_CH0-Pad17) -> /g
- U1 pad 18: unconnected-(U1-GPIO12/ADC2_CH1-Pad18) -> /h
- U1 pad 19: unconnected-(U1-GPIO13/ADC2_CH2-Pad19) -> /i
- U1 pad 20: unconnected-(U1-GPIO14/ADC2_CH3-Pad20) -> /j
- U1 pad 27: unconnected-(U1-GPIO21-Pad27) -> /o
- U1 pad 29: unconnected-(U1-GPIO48-Pad29) -> /LED2?
- U1 pad 32: unconnected-(U1-GPIO35-Pad32) -> /a
- U1 pad 33: unconnected-(U1-GPIO36-Pad33) -> /b
- U1 pad 34: unconnected-(U1-GPIO37-Pad34) -> /c
- U1 pad 35: unconnected-(U1-GPIO38-Pad35) -> /LED1?
- U1 pad 4: unconnected-(U1-GPIO4/ADC1_CH3-Pad4) -> /3
- U1 pad 40: unconnected-(U1-GPIO2/ADC1_CH1-Pad40) -> /2
- U1 pad 41: unconnected-(U1-GPIO1/ADC1_CH0-Pad41) -> /1
- U1 pad 5: unconnected-(U1-GPIO5/ADC1_CH4-Pad5) -> /4
- U1 pad 6: unconnected-(U1-GPIO6/ADC1_CH5-Pad6) -> /5
- U1 pad 7: unconnected-(U1-GPIO7/ADC1_CH6-Pad7) -> /6
- U1 pad 8: unconnected-(U1-GPIO15/ADC2_CH4/32K_P-Pad8) -> /k
- U1 pad 9: unconnected-(U1-GPIO16/ADC2_CH5/32K_N-Pad9) -> /l
Routing:
- net /1: track 270.0 -> 395.2 mm
- net /h: track 198.2 -> 86.1 mm
- net /f: track 196.4 -> 86.1 mm
- net /g: track 197.4 -> 110.0 mm
- net /e: track 147.7 -> 86.1 mm
- net /j: track 206.8 -> 145.9 mm
- net /l: track 87.6 -> 147.6 mm
- net /k: track 87.6 -> 145.2 mm
- net Net-(D42-A): track 6.32 -> 57.1 mm
- net /i: track 188.8 -> 140.4 mm
- net /m: track 86.1 -> 131.0 mm
- net /6: track 323.1 -> 300.0 mm
- net Net-(D73-A): track 6.32 -> 23.7 mm
- net Net-(D74-A): track 6.32 -> 19.0 mm
- net /4: track 262.7 -> 252.4 mm
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Other:
- board size 324.1 x 114.5 mm -> 324.6 x 116.7 mm

Commit message: final hardware
Parts:
- added 3V3: TestPoint, Connector_PinHeader_1.00mm:PinHeader_1x01_P1.00mm_Vertical, F.Cu at (335.3, 29.7)
- added 3V3-2: TestPoint, Connector_PinHeader_1.00mm:PinHeader_1x01_P1.00mm_Vertical, F.Cu at (351.0, 100.8)
- added 5V: TestPoint, Connector_PinHeader_1.00mm:PinHeader_1x01_P1.00mm_Vertical, F.Cu at (338.8, 29.7)
- added 5V-2: TestPoint, Connector_PinHeader_1.00mm:PinHeader_1x01_P1.00mm_Vertical, F.Cu at (351.0, 103.9)
- added GND: TestPoint, Connector_PinHeader_1.00mm:PinHeader_1x01_P1.00mm_Vertical, F.Cu at (342.4, 29.7)
- added GND-2: TestPoint, Connector_PinHeader_1.00mm:PinHeader_1x01_P1.00mm_Vertical, F.Cu at (351.0, 106.9)
- added J3V1: Jumper_2_Open, Jumper:SolderJumper-2_P1.3mm_Open_TrianglePad1.0x1.5mm, F.Cu at (344.4, 88.9)
- added J3V2: Jumper_2_Open, Jumper:SolderJumper-2_P1.3mm_Open_TrianglePad1.0x1.5mm, F.Cu at (344.4, 93.7)
- added J5V1: Jumper_2_Open, Jumper:SolderJumper-2_P1.3mm_Open_TrianglePad1.0x1.5mm, F.Cu at (344.4, 40.6)
- added J5V2: Jumper_2_Open, Jumper:SolderJumper-2_P1.3mm_Open_TrianglePad1.0x1.5mm, F.Cu at (344.4, 38.1)
- added L1: SK6812MINI, kbd:SK6812MINI_rev, B.Cu at (45.2, 100.7)
- added R1: 330R, Resistor_SMD:R_0603_1608Metric_Pad0.98x0.95mm_HandSolder, F.Cu at (333.2, 88.9)
- added R10: 330R, Resistor_SMD:R_0603_1608Metric_Pad0.98x0.95mm_HandSolder, F.Cu at (333.2, 83.8)
- added R11: 330R, Resistor_SMD:R_0603_1608Metric_Pad0.98x0.95mm_HandSolder, F.Cu at (333.2, 76.2)
- added R12: 330R, Resistor_SMD:R_0603_1608Metric_Pad0.98x0.95mm_HandSolder, F.Cu at (333.2, 81.3)
- added R13: 330R, Resistor_SMD:R_0603_1608Metric_Pad0.98x0.95mm_HandSolder, F.Cu at (333.2, 78.7)
- added R14: 330R, Resistor_SMD:R_0603_1608Metric_Pad0.98x0.95mm_HandSolder, F.Cu at (344.4, 61.0)
- added R15: 330R, Resistor_SMD:R_0603_1608Metric_Pad0.98x0.95mm_HandSolder, F.Cu at (344.4, 83.8)
- added R16: 330R, Resistor_SMD:R_0603_1608Metric_Pad0.98x0.95mm_HandSolder, F.Cu at (344.4, 81.3)
- added R17: 330R, Resistor_SMD:R_0603_1608Metric_Pad0.98x0.95mm_HandSolder, F.Cu at (344.4, 78.7)
- added R18: 330R, Resistor_SMD:R_0603_1608Metric_Pad0.98x0.95mm_HandSolder, F.Cu at (344.4, 76.2)
- added R19: 330R, Resistor_SMD:R_0603_1608Metric_Pad0.98x0.95mm_HandSolder, F.Cu at (344.4, 63.5)
- added R2: 330R, Resistor_SMD:R_0603_1608Metric_Pad0.98x0.95mm_HandSolder, F.Cu at (333.2, 86.4)
- added R20: 330R, Resistor_SMD:R_0603_1608Metric_Pad0.98x0.95mm_HandSolder, F.Cu at (344.4, 55.9)
- added R21: 330R, Resistor_SMD:R_0603_1608Metric_Pad0.98x0.95mm_HandSolder, F.Cu at (344.4, 53.3)
- added R22: 330R, Resistor_SMD:R_0603_1608Metric_Pad0.98x0.95mm_HandSolder, F.Cu at (344.4, 50.8)
- added R23: 330R, Resistor_SMD:R_0603_1608Metric_Pad0.98x0.95mm_HandSolder, F.Cu at (344.4, 48.3)
- added R24: 330R, Resistor_SMD:R_0603_1608Metric_Pad0.98x0.95mm_HandSolder, F.Cu at (344.4, 45.7)
- added R25: 330R, Resistor_SMD:R_0603_1608Metric_Pad0.98x0.95mm_HandSolder, F.Cu at (344.4, 43.2)
- added R26: 330R, Resistor_SMD:R_0603_1608Metric_Pad0.98x0.95mm_HandSolder, F.Cu at (344.4, 68.6)
- added R27: 330R, Resistor_SMD:R_0603_1608Metric_Pad0.98x0.95mm_HandSolder, F.Cu at (344.4, 66.0)
- added R28: 330R, Resistor_SMD:R_0603_1608Metric_Pad0.98x0.95mm_HandSolder, F.Cu at (333.2, 48.3)
- added R29: 330R, Resistor_SMD:R_0603_1608Metric_Pad0.98x0.95mm_HandSolder, F.Cu at (333.2, 61.0)
- added R3: 330R, Resistor_SMD:R_0603_1608Metric_Pad0.98x0.95mm_HandSolder, F.Cu at (344.4, 73.7)
- added R30: 330R, Resistor_SMD:R_0603_1608Metric_Pad0.98x0.95mm_HandSolder, F.Cu at (333.2, 63.5)
- added R31: 330R, Resistor_SMD:R_0603_1608Metric_Pad0.98x0.95mm_HandSolder, F.Cu at (333.2, 66.0)
- added R32: 330R, Resistor_SMD:R_0603_1608Metric_Pad0.98x0.95mm_HandSolder, F.Cu at (333.2, 68.6)
- added R33: 330R, Resistor_SMD:R_0603_1608Metric_Pad0.98x0.95mm_HandSolder, F.Cu at (333.2, 55.9)
- added R34: 330R, Resistor_SMD:R_0603_1608Metric_Pad0.98x0.95mm_HandSolder, F.Cu at (344.4, 58.4)
- added R35: 330R, Resistor_SMD:R_0603_1608Metric_Pad0.98x0.95mm_HandSolder, F.Cu at (333.2, 50.8)
- added R36: 330R, Resistor_SMD:R_0603_1608Metric_Pad0.98x0.95mm_HandSolder, F.Cu at (333.2, 53.3)
- added R37: 330R, Resistor_SMD:R_0603_1608Metric_Pad0.98x0.95mm_HandSolder, F.Cu at (344.4, 91.3)
- added R4: 330R, Resistor_SMD:R_0603_1608Metric_Pad0.98x0.95mm_HandSolder, F.Cu at (333.2, 45.7)
- added R5: 330R, Resistor_SMD:R_0603_1608Metric_Pad0.98x0.95mm_HandSolder, F.Cu at (344.4, 71.1)
- added R6: 330R, Resistor_SMD:R_0603_1608Metric_Pad0.98x0.95mm_HandSolder, F.Cu at (333.2, 43.2)
- added R7: 330R, Resistor_SMD:R_0603_1608Metric_Pad0.98x0.95mm_HandSolder, F.Cu at (333.2, 71.1)
- added R8: 330R, Resistor_SMD:R_0603_1608Metric_Pad0.98x0.95mm_HandSolder, F.Cu at (333.2, 58.4)
- added R9: 330R, Resistor_SMD:R_0603_1608Metric_Pad0.98x0.95mm_HandSolder, F.Cu at (333.2, 73.7)
- moved U1 3.80 mm to (350.2, 91.4)
- moved S81 0.06 mm to (342.9, 133.3)
- renumbered D51 to D10, D56 to D11, D62 to D12, D68 to D13, D72 to D14, D77 to D15, D2 to D16, D8 to D17, D14 to D18, D20 to D19, D7 to D2, D26 to D20, D31 to D21, D36 to D22, D41 to D23, D47 to D24, D52 to D25, D57 to D26, D63 to D27, D69 to D28, D75 to D29, D13 to D3, D5 to D30, D11 to D31, D17 to D32, D23 to D33, D28 to D34, D33 to D35, D38 to D36, D44 to D37, D49 to D38, D54 to D39, D19 to D4, D59 to D40, D65 to D41, D70 to D42, D76 to D43, D6 to D44, D12 to D45, D18 to D46, D24 to D47, D29 to D48, D34 to D49, D25 to D5, D39 to D50, D45 to D51, D50 to D52, D55 to D53, D61 to D54, D67 to D55, D74 to D56, D4 to D57, D10 to D58, D16 to D59, D30 to D6, D22 to D60, D27 to D61, D32 to D62, D37 to D63, D43 to D64, D48 to D65, D53 to D66, D58 to D67, D64 to D68, D73 to D69, D35 to D7, D80 to D70, D3 to D71, D9 to D72, D15 to D73, D21 to D74, D42 to D75, D60 to D76, D66 to D77, D71 to D78, D78 to D79, D40 to D8, D79 to D80, D46 to D9, S51 to S10, S56 to S11, S62 to S12, S68 to S13, S72 to S14, S77 to S15, S2 to S16, S8 to S17, S14 to S18, S20 to S19, S7 to S2, S26 to S20, S31 to S21, S36 to S22, S41 to S23, S47 to S24, S52 to S25, S57 to S26, S63 to S27, S69 to S28, S75 to S29, S13 to S3, S5 to S30, S11 to S31, S17 to S32, S23 to S33, S28 to S34, S33 to S35, S38 to S36, S44 to S37, S49 to S38, S54 to S39, S19 to S4, S59 to S40, S65 to S41, S70 to S42, S76 to S43, S6 to S44, S12 to S45, S18 to S46, S24 to S47, S29 to S48, S34 to S49, S25 to S5, S39 to S50, S45 to S51, S50 to S52, S55 to S53, S61 to S54, S67 to S55, S74 to S56, S4 to S57, S10 to S58, S16 to S59, S30 to S6, S22 to S60, S27 to S61, S32 to S62, S37 to S63, S43 to S64, S48 to S65, S53 to S66, S58 to S67, S64 to S68, S73 to S69, S35 to S7, S79 to S70, S3 to S71, S9 to S72, S15 to S73, S21 to S74, S42 to S75, S60 to S76, S66 to S77, S71 to S78, S78 to S79, S40 to S8, S46 to S9
Connections:
- net Net-(U1-3V3-Pad1) renamed +3.3V
- net Net-(U1-GND-Pad22) renamed GND
- U1 pad 10: /m -> Net-(U1-GPIO17/ADC2_CH6)
- U1 pad 11: /n -> Net-(U1-GPIO18/ADC2_CH7)
- U1 pad 12: /d -> Net-(U1-GPIO8/ADC1_CH7)
- U1 pad 13: unconnected-(U1-GPIO3/ADC1_CH2-Pad13) -> Net-(U1-GPIO3/ADC1_CH2)
- U1 pad 14: unconnected-(U1-GPIO46-Pad14) -> Net-(U1-GPIO46)
- U1 pad 15: /e -> Net-(U1-GPIO9/ADC1_CH8)
- U1 pad 16: /f -> Net-(U1-GPIO10/ADC1_CH9)
- U1 pad 17: /g -> Net-(U1-GPIO11/ADC2_CH0)
- U1 pad 18: /h -> Net-(U1-GPIO12/ADC2_CH1)
- U1 pad 19: /i -> Net-(U1-GPIO13/ADC2_CH2)
- U1 pad 20: /j -> Net-(U1-GPIO14/ADC2_CH3)
- U1 pad 21: unconnected-(U1-5V-Pad21) -> +5V
- U1 pad 25: unconnected-(U1-GPIO19/USB_D--Pad25) -> Net-(U1-GPIO19/USB_D-)
- U1 pad 26: unconnected-(U1-GPIO20/USB_D+-Pad26) -> Net-(U1-GPIO20/USB_D+)
- U1 pad 27: /o -> Net-(U1-GPIO21)
- U1 pad 28: unconnected-(U1-GPIO47-Pad28) -> Net-(U1-GPIO47)
- U1 pad 30: unconnected-(U1-GPIO45-Pad30) -> Net-(U1-GPIO45)
- U1 pad 31: unconnected-(U1-GPIO0-Pad31) -> Net-(U1-GPIO0)
- U1 pad 32: /a -> Net-(U1-GPIO35)
- U1 pad 33: /b -> Net-(U1-GPIO36)
- U1 pad 34: /c -> Net-(U1-GPIO37)
- U1 pad 36: unconnected-(U1-GPIO39/MTCK-Pad36) -> Net-(U1-GPIO39/MTCK)
- U1 pad 37: unconnected-(U1-GPIO40/MTDO-Pad37) -> Net-(U1-GPIO40/MTDO)
- U1 pad 38: unconnected-(U1-GPIO41/MTDI-Pad38) -> Net-(U1-GPIO41/MTDI)
- U1 pad 39: unconnected-(U1-GPIO42/MTMS-Pad39) -> Net-(U1-GPIO42/MTMS)
- U1 pad 4: /3 -> Net-(U1-GPIO4/ADC1_CH3)
- U1 pad 40: /2 -> Net-(U1-GPIO2/ADC1_CH1)
- U1 pad 41: /1 -> Net-(U1-GPIO1/ADC1_CH0)
- U1 pad 42: unconnected-(U1-GPIO44/U0RXD-Pad42) -> Net-(U1-GPIO44/U0RXD)
- U1 pad 43: unconnected-(U1-GPIO43/U0TXD-Pad43) -> Net-(U1-GPIO43/U0TXD)
- U1 pad 5: /4 -> Net-(U1-GPIO5/ADC1_CH4)
- U1 pad 6: /5 -> Net-(U1-GPIO6/ADC1_CH5)
- U1 pad 7: /6 -> Net-(U1-GPIO7/ADC1_CH6)
- U1 pad 8: /k -> Net-(U1-GPIO15/ADC2_CH4/32K_P)
- U1 pad 9: /l -> Net-(U1-GPIO16/ADC2_CH5/32K_N)
Routing:
- net /CAPS_LED: track 0.00 -> 329.2 mm, vias 0 -> 2
- net Net-(L1-VDD): track 0.00 -> 319.4 mm, vias 0 -> 2
- net /a: track 100.2 -> 408.5 mm, vias 0 -> 1
- net /b: track 105.1 -> 407.0 mm, vias 0 -> 1
- net /c: track 105.1 -> 380.4 mm, vias 0 -> 1
- net /e: track 86.1 -> 360.9 mm, vias 0 -> 1
- net /f: track 86.1 -> 336.1 mm, vias 0 -> 1
- net /d: track 105.1 -> 355.1 mm, vias 0 -> 1
- net /g: track 110.0 -> 340.6 mm, vias 0 -> 1
- net /h: track 86.1 -> 295.4 mm, vias 0 -> 1
- net /i: track 140.4 -> 328.5 mm, vias 0 -> 1
- net /j: track 145.9 -> 312.8 mm, vias 0 -> 1
- net /k: track 145.2 -> 285.8 mm, vias 0 -> 1
- net /l: track 147.6 -> 266.9 mm, vias 0 -> 1
- net /m: track 131.0 -> 229.2 mm, vias 0 -> 1
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- added copper zone on B.Cu, net GND
- added copper zone on F.Cu, net GND
Other:
- board text added: "JLCJLCJLCJLC"
